Commit message: chore: added first approach urdf

File: waver_ws/src/waver_description/urdf/waver.urdf (robot description, URDF)
Before this commit: robot my_robot, 1 links, 0 joints
Links:
- added link top_shell_link, mass 0.5; collision box size=0.5 0.3 0.02; visual box size=0.5 0.3 0.02
- link base_link: mass None -> 1.0; geometry collision box size=0.5 0.3 0.02; visual box size=0.5 0.3 0.02
Joints:
- added joint base_to_top: type fixed, parent base_link, child top_shell_link, origin xyz=0 0 0.1 rpy=0 0 0

Commit message: fix: tf issues with wheels

File: waver_ws/src/waver_description/urdf/waver.urdf (robot description, URDF)
Before this commit: robot waver, 2 links, 1 joints
Links:
- added link dummy_link, mass 0.01; collision box size=0.01 0.01 0.01; visual box size=0.01 0.01 0.01
Joints:
- added joint dummy_to_base: type fixed, parent dummy_link, child base_link, origin xyz=0 0 0 rpy=0 0 0

File: waver_ws/src/waver_description/urdf/waver.xacro (robot description, xacro)
@@ -19,5 +19,5 @@
             </inertial>
         </link>
-        <joint name="${name}_joint" type="continuous">
+        <joint name="${name}_joint" type="fixed">
             <parent link="base_link" />
             <child link="${name}" />

Commit message: chore: improve global frame with tf2

File: waver_ws/src/waver_description/urdf/waver.urdf (robot description, URDF)
Before this commit: robot waver, 3 links, 2 joints
Links:
- removed link dummy_link
- added link base_footprint, mass 0.01; collision box size=0.001 0.001 0.001; visual box size=0.001 0.001 0.001
Joints:
- removed joint dummy_to_base
- added joint base_joint: type fixed, parent base_footprint, child base_link, origin xyz=0 0 0.135 rpy=0 0 0

Commit message: chore: improvement compilation and testing

File: waver_ws/src/waver_description/urdf/waver.urdf (robot description, URDF)
Before this commit: robot waver, 3 links, 2 joints
Links:
- link base_footprint: mass 0.01 -> None; geometry visual box size=0.01 0.01 0.01

File: waver_ws/src/waver_description/urdf/waver.xacro (robot description, xacro)
@@ -5,10 +5,13 @@
             <visual>
                 <geometry>
-                    <cylinder length="0.05" radius="0.1" />
+                    <cylinder length="0.1" radius="0.1" />
                 </geometry>
+                <material name="black">
+                    <color rgba="0 0 0 1" />
+                </material>
             </visual>
             <collision>
                 <geometry>
-                    <cylinder length="0.05" radius="0.1" />
+                    <cylinder length="0.1" radius="0.1" />
                 </geometry>
             </collision>
@@ -19,5 +22,5 @@
             </inertial>
         </link>
-        <joint name="${name}_joint" type="fixed">
+        <joint name="${name}_joint" type="continuous">
             <parent link="base_link" />
             <child link="${name}" />

Commit message: chore: implemented meshes launch rviz and gazebo (first approach)

File: waver_ws/src/waver_description/urdf/waver.urdf (robot description, URDF)
Before this commit: robot waver, 3 links, 2 joints
Links:
- link base_footprint: geometry 
- link base_link: mass 1.0 -> 0.6; geometry collision box size=0.5 0.3 0.02; visual mesh filename=package://waver_description/meshes/base_link_husky.stl scale=1 1 1
- link top_shell_link: geometry collision box size=0.5 0.3 0.02; visual mesh filename=package://waver_description/meshes/top_plate_husky.stl scale=0.8 0.8 0.8
Joints:
- removed joint base_to_top
- added joint base_to_top_joint: type fixed, parent base_link, child top_shell_link, origin xyz=0 0 0.225 rpy=0 0 0
- joint base_joint: origin xyz=0 0 0.135 rpy=0 0 0 -> xyz=0 0 0.16 rpy=0 0 0

File: waver_ws/src/waver_description/urdf/waver.xacro (robot description, xacro)
@@ -2,8 +2,8 @@
 <robot xmlns:xacro="http://www.ros.org/wiki/xacro" name="waver">
     <xacro:macro name="wheel" params="name xyz rpy">
-        <link name="${name}">
+        <link name="${name}_link">
             <visual>
                 <geometry>
-                    <cylinder length="0.1" radius="0.1" />
+                    <mesh filename="package://waver_description/meshes/wheel_husky.stl" scale="1 1 1"/>
                 </geometry>
                 <material name="black">
@@ -24,5 +24,5 @@
         <joint name="${name}_joint" type="continuous">
             <parent link="base_link" />
-            <child link="${name}" />
+            <child link="${name}_link" />
             <origin xyz="${xyz}" rpy="${rpy}" />
             <axis xyz="0 0 1" />

Commit message: refactor: refactoring urdf files | improved values

File: waver_ws/src/waver_description/urdf/waver.urdf (robot description, URDF)
Before this commit: robot waver, 3 links, 2 joints
Links:
- link base_link: mass 0.6 -> ${base_mass}; geometry collision mesh filename=package://waver_description/meshes/base_link_husky.stl scale=1 1 1; visual mesh filename=package://waver_description/meshes/base_link_husky.stl scale=1 1 1
- link top_shell_link: mass 0.5 -> ${top_mass}; geometry collision mesh filename=package://waver_description/meshes/top_plate_husky.stl scale=1 1 1; visual mesh filename=package://waver_description/meshes/top_plate_husky.stl scale=1 1 1
Joints:
- joint base_joint: origin xyz=0 0 0.16 rpy=0 0 0 -> xyz=0 0 ${-(0.03282-0.1651)} rpy=0 0 0
