Commit message: feat: gazebo implementation | inertia improvement

File: waver_ws/src/waver_description/urdf/inertial_wheel.xacro (robot description, xacro)
@@ -6,5 +6,5 @@
             <mass value="${wheel_mass}" />
             <origin xyz="${triple_zero}" rpy="${triple_zero}" />
-            <inertia ixx="${I_wheel}" ixy="0" ixz="0" iyy="${I_wheel}" iyz="0" izz="${Iz_wheel}" />
+            <inertia  ixx="${Ixx_wheel}" ixy="0" ixz="0" iyy="${Iyy_wheel}" iyz="0" izz="${Izz_wheel}" />
         </inertial>
     </xacro:macro>

File: waver_ws/src/waver_description/urdf/util.xacro (robot description, xacro)
@@ -6,13 +6,26 @@
     <xacro:property name="wheel_radius" value="0.1651" />
     <xacro:property name="wheel_length" value="0.1143" />
-    <xacro:property name="wheel_mass" value="0.5" />
-    <xacro:property name="Iz_wheel" value="${0.5*wheel_mass*wheel_radius*wheel_radius}" />
-    <xacro:property name="I_wheel" value="${-(1/12)*wheel_mass*(3*wheel_radius*wheel_radius+wheel_length*wheel_length)}" />
+    <xacro:property name="wheel_mass" value="2.637" />
+    <xacro:property name="Ixx_wheel" value="0.02467" />
+    <xacro:property name="Iyy_wheel" value="0.04411" />
+    <xacro:property name="Izz_wheel" value="0.02467" />
     <!-- Base link specifications -->
-    <xacro:property name="base_mass" value="0.75" />
-    <xacro:property name="base_x_len" value="0.5120" />
-    <xacro:property name="base_y_len" value="0.5708" />
-    <xacro:property name="base_h_len" value="0.03282" />
+    <xacro:property name="base_length" value="0.71" />
+    <xacro:property name="base_width" value="0.41" />
+    <xacro:property name="base_thickness" value="0.025" />
+    <xacro:property name="base_mass" value="6.0" />
+    <xacro:property name="Ixx_base" value="${(base_mass/12) * (base_length * base_length + base_width * base_width)}" />
+    <xacro:property name="Iyy_base" value="${(base_mass/12) * (base_length * base_length + base_thickness * base_thickness)}" />
+    <xacro:property name="Izz_base" value="${(base_mass/12) * (base_width * base_width + base_thickness * base_thickness)}" />
+    <xacro:property name="base_x" value="0.5120" />
+    <xacro:property name="base_y" value="0.5708" />
+    <xacro:property name="base_h" value="0.03282" />
     <!-- Top shell specifications -->
-    <xacro:property name="top_mass" value="0.5" />
+    <xacro:property name="top_length" value="0.725" />
+    <xacro:property name="top_width" value="0.59" />
+    <xacro:property name="top_thickness" value="0.006" />
+    <xacro:property name="top_mass" value="2.5" />
+    <xacro:property name="Ixx_top" value="${(top_mass/12) * (top_length * top_length + top_width * top_width)}" />
+    <xacro:property name="Iyy_top" value="${(top_mass/12) * (top_length * top_length + top_thickness * top_thickness)}" />
+    <xacro:property name="Izz_top" value="${(top_mass/12) * (top_width * top_width + top_thickness * top_thickness)}" />
 </robot>

File: waver_ws/src/waver_description/urdf/waver.urdf (robot description, URDF)
Before this commit: robot waver, 3 links, 2 joints
Joints:
- joint base_joint: origin xyz=0 0 ${-(0.03282-0.1651)} rpy=0 0 0 -> xyz=0 0 ${-(base_h - wheel_radius)} rpy=0 0 0

File: waver_ws/src/waver_description/urdf/wheel.xacro (robot description, xacro)
@@ -1,12 +1,12 @@
 <?xml version="1.0"?>
 <robot xmlns:xacro="http://www.ros.org/wiki/xacro" name="wheels">
-    <xacro:include filename="$(find waver_description)/urdf/materials.xacro"/>
+    <xacro:include filename="$(find waver_description)/urdf/materials.xacro" />
     <xacro:include filename="$(find waver_description)/urdf/inertial_wheel.xacro" />
+    <xacro:include filename="$(find waver_description)/urdf/util.xacro" />
     <xacro:macro name="wheel" params="prefix suffix xyz rpy">
         <link name="${prefix}_${suffix}_link">
             <visual>
                 <geometry>
-                    <mesh filename="package://waver_description/meshes/wheel_husky.stl"
-                        scale="1 1 1" />
+                    <mesh filename="package://waver_description/meshes/wheel_husky.stl" scale="1 1 1" />
                 </geometry>
                 <xacro:black_material />
@@ -14,6 +14,5 @@
             <collision>
                 <geometry>
-                    <mesh filename="package://waver_description/meshes/wheel_husky.stl"
-                        scale="1 1 1" />
+                    <mesh filename="package://waver_description/meshes/wheel_husky.stl" scale="1 1 1" />
                 </geometry>
             </collision>
@@ -27,15 +26,18 @@
         </joint>
         <transmission name="${prefix}_${suffix}_wheel_trans" type="SimpleTransmission">
-			<type>transmission_interface/SimpleTransmission</type>
-			<actuator name="${prefix}_${suffix}_wheel_motor">
-				<mechanicalReduction>1</mechanicalReduction>
-			</actuator>
-			<joint name="${prefix}_${suffix}_joint">
-				<hardwareInterface>hardware_interface/VelocityJointInterface</hardwareInterface>
-			</joint>
-		</transmission>
+            <type>transmission_interface/SimpleTransmission</type>
+            <actuator name="${prefix}_${suffix}_wheel_motor">
+                <mechanicalReduction>1</mechanicalReduction>
+            </actuator>
+            <joint name="${prefix}_${suffix}_joint">
+                <hardwareInterface>hardware_interface/VelocityJointInterface</hardwareInterface>
+            </joint>
+        </transmission>
         <gazebo reference="${prefix}_${suffix}_link">
-            <mu1 value="0.1" />
-            <mu2 value="0.1" />
+            <mu1 value="1.0" />
+            <mu2 value="1.0" />
+            <kp value="100000.0" />
+            <kd value="10.0" />
+            <fdir1 value="1 0 0" />
             <material>Gazebo/Black</material>
         </gazebo>
