Commit message: feat: waver description using fusion360

File: waver_ws/src/waver_description/urdf/materials.xacro (robot description, xacro)
@@ -1,7 +1,12 @@
 <?xml version="1.0"?>
-<robot xmlns:xacro="http://ros.org/wiki/xacro" name="material_definitions">
-    <xacro:macro name="gray_material">
-        <material name="gray">
-            <color rgba="0.5 0.5 0.5 1" />
+<robot xmlns:xacro="http://ros.org/wiki/xacro" name="waver_material">
+    <xacro:macro name="dark_gray_material">
+        <material name="_dark_gray">
+            <color rgba="0.4 0.4 0.4 1" />
+        </material>
+    </xacro:macro>
+    <xacro:macro name="light_gray_material">
+        <material name="light_gray">
+            <color rgba="0.6 0.6 0.6 1" />
         </material>
     </xacro:macro>
@@ -16,3 +21,13 @@
         </material>
     </xacro:macro>
+    <xacro:macro name="dark_green_material">
+        <material name="dark_green">
+            <color rgba="0.86 0.625 0.52 1" />
+        </material>
+    </xacro:macro>
+    <xacro:macro name="dark_blue_material">
+        <material name="dark_blue">
+            <color rgba="0.0156 0.23 0.4 1" />
+        </material>
+    </xacro:macro>
 </robot>

File: waver_ws/src/waver_description/urdf/util.xacro (robot description, xacro)
@@ -1,31 +1,7 @@
 <?xml version="1.0"?>
-<robot xmlns:xacro="http://www.ros.org/wiki/xacro" name="utils">
+<robot xmlns:xacro="http://www.ros.org/wiki/xacro" name="waver_utils">
     <xacro:property name="triple_zero" value="0 0 0" />
+    <xacro:property name="scale" value="0.001 0.001 0.001" />
     <xacro:property name="pi" value="3.14159265" />
     <!-- Wheel specifications -->
-    <xacro:property name="wheel_radius" value="0.1651" />
-    <xacro:property name="wheel_length" value="0.1143" />
-    <xacro:property name="wheel_mass" value="2.637" />
-    <xacro:property name="Ixx_wheel" value="0.02467" />
-    <xacro:property name="Iyy_wheel" value="0.04411" />
-    <xacro:property name="Izz_wheel" value="0.02467" />
-    <!-- Base link specifications -->
-    <xacro:property name="base_length" value="0.71" />
-    <xacro:property name="base_width" value="0.41" />
-    <xacro:property name="base_thickness" value="0.025" />
-    <xacro:property name="base_mass" value="6.0" />
-    <xacro:property name="Ixx_base" value="${(base_mass/12) * (base_length * base_length + base_width * base_width)}" />
-    <xacro:property name="Iyy_base" value="${(base_mass/12) * (base_length * base_length + base_thickness * base_thickness)}" />
-    <xacro:property name="Izz_base" value="${(base_mass/12) * (base_width * base_width + base_thickness * base_thickness)}" />
-    <xacro:property name="base_x" value="0.5120" />
-    <xacro:property name="base_y" value="0.5708" />
-    <xacro:property name="base_h" value="0.03282" />
-    <!-- Top shell specifications -->
-    <xacro:property name="top_length" value="0.725" />
-    <xacro:property name="top_width" value="0.59" />
-    <xacro:property name="top_thickness" value="0.006" />
-    <xacro:property name="top_mass" value="2.5" />
-    <xacro:property name="Ixx_top" value="${(top_mass/12) * (top_length * top_length + top_width * top_width)}" />
-    <xacro:property name="Iyy_top" value="${(top_mass/12) * (top_length * top_length + top_thickness * top_thickness)}" />
-    <xacro:property name="Izz_top" value="${(top_mass/12) * (top_width * top_width + top_thickness * top_thickness)}" />
 </robot>
