Commit message: chore: improvement transmissions | links specifications | gazebo env

File: waver_ws/src/waver_description/urdf/util.xacro (robot description, xacro)
@@ -4,4 +4,76 @@
     <xacro:property name="scale" value="0.001 0.001 0.001" />
     <xacro:property name="pi" value="3.14159265" />
-    <!-- Wheel specifications -->
+    <!-- Base specifications -->
+    <xacro:property name="pos_x_base" value="2.838767506182194e-05" />
+    <xacro:property name="pos_y_base" value="-6.582658272236586e-06" />
+    <xacro:property name="pos_z_base" value="0.002703800678253174" />
+    <xacro:property name="mass_base" value="0.37038398045076265" />
+    <xacro:property name="mass_center_base" value="${pos_x_base} ${pos_y_base} ${pos_z_base}" />
+    <xacro:property name="position_base" value="${-pos_x_base} ${-pos_y_base} ${-pos_z_base}" />
+    <!-- Top specifications -->
+    <xacro:property name="pos_x_top" value="0.00018196851015090943" />
+    <xacro:property name="pos_y_top" value="-0.0006833337545394898" />
+    <xacro:property name="pos_z_top" value="0.038709537506103515" />
+    <xacro:property name="mass_top" value="0.7277708834628859" />
+    <xacro:property name="mass_center_top" value="${pos_x_top} ${pos_y_top} ${pos_z_top}" />
+    <xacro:property name="position_top" value="${-pos_x_top} ${-pos_y_top} ${-pos_z_top}" />
+    <!-- Accessories specifications -->
+    <xacro:property name="pos_x_acces" value="-0.02246641731262207" />
+    <xacro:property name="pos_y_acces" value="0.08693458557128907" />
+    <xacro:property name="pos_z_acces" value="0.04861989974975586" />
+    <xacro:property name="mass_acces" value="0.017616158924187116" />
+    <xacro:property name="mass_center_acces" value="${pos_x_acces} ${pos_y_acces} ${pos_z_acces}" />
+    <xacro:property name="position_acces" value="${-pos_x_acces} ${-pos_y_acces} ${-pos_z_acces}" />
+    <!-- Accessories1 specifications -->
+    <xacro:property name="pos_x_acces1" value="-0.002510018587112427" />
+    <xacro:property name="pos_y_acces1" value="0.07360986328125002" />
+    <xacro:property name="pos_z_acces1" value="0.035275302886962887" />
+    <xacro:property name="mass_acces1" value="0.021489822783274555" />
+    <xacro:property name="mass_center_acces1" value="${pos_x_acces1} ${pos_y_acces1} ${pos_z_acces1}" />
+    <xacro:property name="position_acces1" value="${-pos_x_acces1} ${-pos_y_acces1} ${-pos_z_acces1}" />
+    <!-- Board speficications -->
+    <xacro:property name="pos_x_board" value="-0.009815516471862793" />
+    <xacro:property name="pos_y_board" value="0.009279213905334474" />
+    <xacro:property name="pos_z_board" value="0.04129100418090821" />
+    <xacro:property name="mass_board" value="0.12365568710683028" />
+    <xacro:property name="mass_center_board" value="${pos_x_board} ${pos_y_board} ${pos_z_board}" />
+    <xacro:property name="position_board" value="${-pos_x_board} ${-pos_y_board} ${-pos_z_board}" />
+    <!-- Oled Screen speficications -->
+    <xacro:property name="pos_x_screen" value="-6.735318456776441e-07" />
+    <xacro:property name="pos_y_screen" value="0.05096461868286133" />
+    <xacro:property name="pos_z_screen" value="0.048232952117919926" />
+    <xacro:property name="mass_screen" value="0.014091265350616076" />
+    <xacro:property name="mass_center_screen" value="${pos_x_screen} ${pos_y_screen} ${pos_z_screen}" />
+    <xacro:property name="position_screen" value="${-pos_x_screen} ${-pos_y_screen} ${-pos_z_screen}" />
+    <!-- Wheels specifications -->
+    <xacro:property name="wheel_separation" value="123e-3" />
+    <xacro:property name="wheel_radius" value="40.6e-3" />
+    <!-- WBL specifications -->
+    <xacro:property name="pos_x_wbl" value="0.06538582611083985" />
+    <xacro:property name="pos_y_wbl" value="0.04859128189086914" />
+    <xacro:property name="pos_z_wbl" value="0.004798986434936523" />
+    <xacro:property name="mass_wbl" value="1.01701435808657" />
+    <xacro:property name="mass_center_wbl" value="${pos_x_wbl} ${pos_y_wbl} ${pos_z_wbl}" />
+    <xacro:property name="position_wbl" value="${-pos_x_wbl} ${-pos_y_wbl} ${-pos_z_wbl}" />
+    <!-- WFL specifications -->
+    <xacro:property name="pos_x_wfl" value="0.06538582611083985" />
+    <xacro:property name="pos_y_wfl" value="-0.048406845092773446" />
+    <xacro:property name="pos_z_wfl" value="0.004799012184143066" />
+    <xacro:property name="mass_wfl" value="1.0170155374515382" />
+    <xacro:property name="mass_center_wfl" value="${pos_x_wfl} ${pos_y_wfl} ${pos_z_wfl}" />
+    <xacro:property name="position_wfl" value="${-pos_x_wfl} ${-pos_y_wfl} ${-pos_z_wfl}" />
+    <!-- WFR specifications -->
+    <xacro:property name="pos_x_wfr" value="-0.06528724670410156" />
+    <xacro:property name="pos_y_wfr" value="-0.048593093872070316" />
+    <xacro:property name="pos_z_wfr" value="0.004798998355865478" />
+    <xacro:property name="mass_wfr" value="1.0170112199417978" />
+    <xacro:property name="mass_center_wfr" value="${pos_x_wfr} ${pos_y_wfr} ${pos_z_wfr}" />
+    <xacro:property name="position_wfr" value="${-pos_x_wfr} ${-pos_y_wfr} ${-pos_z_wfr}" />
+    <!-- WBR specifications -->
+    <xacro:property name="pos_x_wbr" value="-0.0652872543334961" />
+    <xacro:property name="pos_y_wbr" value="0.04840502166748047" />
+    <xacro:property name="pos_z_wbr" value="0.004799028396606446" />
+    <xacro:property name="mass_wbr" value="1.0170123141691128" />
+    <xacro:property name="mass_center_wbr" value="${pos_x_wbr} ${pos_y_wbr} ${pos_z_wbr}" />
+    <xacro:property name="position_wbr" value="${-pos_x_wbr} ${-pos_y_wbr} ${-pos_z_wbr}" />
 </robot>

File: waver_ws/src/waver_description/urdf/waver.gazebo.xacro (robot description, xacro)
@@ -1,12 +1,12 @@
 <?xml version="1.0"?>
 <robot xmlns:xacro="http://www.ros.org/wiki/xacro" name="waver_gazebo">
-  <gazebo>
+  <xacro:include filename="$(find waver_description)/urdf/util.xacro" />
+  <!-- <gazebo>
     <plugin name="control" filename="libgazebo_ros_control.so" />
-  </gazebo>
+  </gazebo> -->
   <gazebo reference="base_link">
     <mu1>0.2</mu1>
     <mu2>0.2</mu2>
-    <selfCollide>true</selfCollide>
-    <gravity>true</gravity>
+    <selfCollide>false</selfCollide>
     <material>Gazebo/DarkGrey</material>
   </gazebo>
@@ -14,5 +14,5 @@
     <mu1>0.2</mu1>
     <mu2>0.2</mu2>
-    <selfCollide>true</selfCollide>
+    <selfCollide>false</selfCollide>
     <material>Gazebo/DarkGrey</material>
   </gazebo>
@@ -20,5 +20,5 @@
     <mu1>0.2</mu1>
     <mu2>0.2</mu2>
-    <selfCollide>true</selfCollide>
+    <selfCollide>false</selfCollide>
     <material>Gazebo/Black</material>
   </gazebo>
@@ -26,5 +26,5 @@
     <mu1>0.2</mu1>
     <mu2>0.2</mu2>
-    <selfCollide>true</selfCollide>
+    <selfCollide>false</selfCollide>
     <material>Gazebo/Black</material>
   </gazebo>
@@ -32,5 +32,5 @@
     <mu1>0.2</mu1>
     <mu2>0.2</mu2>
-    <selfCollide>true</selfCollide>
+    <selfCollide>false</selfCollide>
     <material>Gazebo/Orange</material>
   </gazebo>
@@ -38,5 +38,5 @@
     <mu1>0.2</mu1>
     <mu2>0.2</mu2>
-    <selfCollide>true</selfCollide>
+    <selfCollide>false</selfCollide>
     <material>Gazebo/BlueGlow</material>
   </gazebo>
@@ -44,5 +44,5 @@
     <mu1>0.2</mu1>
     <mu2>0.2</mu2>
-    <selfCollide>true</selfCollide>
+    <selfCollide>false</selfCollide>
     <material>Gazebo/Black</material>
   </gazebo>
@@ -50,5 +50,5 @@
     <mu1>0.2</mu1>
     <mu2>0.2</mu2>
-    <selfCollide>true</selfCollide>
+    <selfCollide>false</selfCollide>
     <material>Gazebo/Black</material>
   </gazebo>
@@ -56,5 +56,5 @@
     <mu1>0.2</mu1>
     <mu2>0.2</mu2>
-    <selfCollide>true</selfCollide>
+    <selfCollide>false</selfCollide>
     <material>Gazebo/Black</material>
   </gazebo>
@@ -62,5 +62,5 @@
     <mu1>0.2</mu1>
     <mu2>0.2</mu2>
-    <selfCollide>true</selfCollide>
+    <selfCollide>false</selfCollide>
     <material>Gazebo/Black</material>
   </gazebo>

File: waver_ws/src/waver_description/urdf/waver.trans.xacro (robot description, xacro)
@@ -1,41 +1,41 @@
 <?xml version="1.0"?>
 <robot xmlns:xacro="http://www.ros.org/wiki/xacro" name="waver_transmission">
-  <transmission name="base_wbl_joint_tran">
+  <transmission name="wheel_back_left_joint_tran" type="SimpleTransmission">
     <type>transmission_interface/SimpleTransmission</type>
-    <joint name="base_wbl_joint">
-      <hardwareInterface>hardware_interface/EffortJointInterface</hardwareInterface>
+    <joint name="wheel_back_left_joint">
+      <hardwareInterface>hardware_interface/VelocityJointInterface</hardwareInterface>
     </joint>
-    <actuator name="base_wbl_joint_actr">
-      <hardwareInterface>hardware_interface/EffortJointInterface</hardwareInterface>
+    <actuator name="wheel_back_left_joint_actr">
+      <hardwareInterface>hardware_interface/VelocityJointInterface</hardwareInterface>
       <mechanicalReduction>1</mechanicalReduction>
     </actuator>
   </transmission>
-  <transmission name="base_wfl_joint_tran">
+  <transmission name="wheel_front_left_joint_tran">
     <type>transmission_interface/SimpleTransmission</type>
-    <joint name="base_wfl_joint">
-      <hardwareInterface>hardware_interface/EffortJointInterface</hardwareInterface>
+    <joint name="wheel_front_left_joint">
+      <hardwareInterface>hardware_interface/VelocityJointInterface</hardwareInterface>
     </joint>
-    <actuator name="base_wfl_joint_actr">
-      <hardwareInterface>hardware_interface/EffortJointInterface</hardwareInterface>
+    <actuator name="wheel_front_left_joint_actr">
+      <hardwareInterface>hardware_interface/VelocityJointInterface</hardwareInterface>
       <mechanicalReduction>1</mechanicalReduction>
     </actuator>
   </transmission>
-  <transmission name="base_wfr_joint_tran">
+  <transmission name="wheel_front_right_joint_tran">
     <type>transmission_interface/SimpleTransmission</type>
-    <joint name="base_wfr_joint">
-      <hardwareInterface>hardware_interface/EffortJointInterface</hardwareInterface>
+    <joint name="wheel_front_right_joint">
+      <hardwareInterface>hardware_interface/VelocityJointInterface</hardwareInterface>
     </joint>
-    <actuator name="base_wfr_joint_actr">
-      <hardwareInterface>hardware_interface/EffortJointInterface</hardwareInterface>
+    <actuator name="wheel_front_right_joint_actr">
+      <hardwareInterface>hardware_interface/VelocityJointInterface</hardwareInterface>
       <mechanicalReduction>1</mechanicalReduction>
     </actuator>
   </transmission>
-  <transmission name="base_wbr_joint_tran">
+  <transmission name="wheel_back_right_joint_tran">
     <type>transmission_interface/SimpleTransmission</type>
-    <joint name="base_wbr_joint">
-      <hardwareInterface>hardware_interface/EffortJointInterface</hardwareInterface>
+    <joint name="wheel_back_right_joint">
+      <hardwareInterface>hardware_interface/VelocityJointInterface</hardwareInterface>
     </joint>
-    <actuator name="base_wbr_joint_actr">
-      <hardwareInterface>hardware_interface/EffortJointInterface</hardwareInterface>
+    <actuator name="wheel_back_right_joint_actr">
+      <hardwareInterface>hardware_interface/VelocityJointInterface</hardwareInterface>
       <mechanicalReduction>1</mechanicalReduction>
     </actuator>

File: waver_ws/src/waver_description/urdf/waver.xacro (robot description, xacro)
@@ -9,6 +9,6 @@
   <link name="base_link">
     <inertial>
-      <mass value="0.37038398045076265" />
-      <origin xyz="2.838767506182194e-05 -6.582658272236586e-06 0.002703800678253174" rpy="0 0 0" />
+      <mass value="${mass_base}" />
+      <origin xyz="${mass_center_base}" rpy="0 0 0" />
       <inertia ixx="8.590754" iyy="4.272701" izz="12.732361" ixy="-0.00783" iyz="-1.6e-05" ixz="-0.000187" />
     </inertial>
@@ -29,6 +29,6 @@
   <link name="top_shell_link">
     <inertial>
-      <mass value="0.7277708834628859" />
-      <origin xyz="0.00018196851015090943 -0.0006833337545394898 0.038709537506103515" rpy="0 0 0" />
+      <mass value="${mass_top}" />
+      <origin xyz="${mass_center_top}" rpy="0 0 0" />
       <inertia ixx="23.275057" iyy="12.620651" izz="32.42524" ixy="-0.009322" iyz="0.010328" ixz="-0.015376" />
     </inertial>
@@ -49,10 +49,10 @@
   <link name="accessories_link">
     <inertial>
-      <mass value="0.017616158924187116" />
-      <origin xyz="-0.02246641731262207 0.08693458557128907 0.04861989974975586" rpy="0 0 0" />
+      <mass value="${mass_acces}" />
+      <origin xyz="${mass_center_acces}" rpy="0 0 0" />
       <inertia ixx="0.015855" iyy="0.037389" izz="0.037412" ixy="0.00687" iyz="-0.007022" ixz="0.006879" />
     </inertial>
     <visual>
-      <origin xyz="0 0 0" rpy="0 0 0" />
+      <origin xyz="${position_acces}" rpy="0 0 0" />
       <geometry>
         <mesh filename="package://waver_description/meshes/accessories_link.stl" scale="${scale}" />
@@ -61,5 +61,5 @@
     </visual>
     <collision>
-      <origin xyz="0 0 0" rpy="0 0 0" />
+      <origin xyz="${position_acces}" rpy="0 0 0" />
       <geometry>
         <mesh filename="package://waver_description/meshes/accessories_link.stl" scale="${scale}" />
@@ -69,10 +69,10 @@
   <link name="accessories1_link">
     <inertial>
-      <mass value="0.021489822783274555" />
-      <origin xyz="-0.002510018587112427 0.07360986328125002 0.035275302886962887" rpy="0 0 0" />
+      <mass value="${mass_acces1}" />
+      <origin xyz="${mass_center_acces1}" rpy="0 0 0" />
       <inertia ixx="0.008308" iyy="0.027844" izz="0.02786" ixy="0.000652" iyz="-0.002643" ixz="0.000591" />
     </inertial>
     <visual>
-      <origin xyz="0 0 0" rpy="0 0 0" />
+      <origin xyz="${position_acces1}" rpy="0 0 0" />
       <geometry>
         <mesh filename="package://waver_description/meshes/accessories1_link.stl" scale="${scale}" />
@@ -81,5 +81,5 @@
     </visual>
     <collision>
-      <origin xyz="0 0 0" rpy="0 0 0" />
+      <origin xyz="${position_acces1}" rpy="0 0 0" />
       <geometry>
         <mesh filename="package://waver_description/meshes/accessories1_link.stl" scale="${scale}" />
@@ -89,10 +89,10 @@
   <link name="board_link">
     <inertial>
-      <mass value="0.12365568710683028" />
-      <origin xyz="-0.009815516471862793 0.009279213905334474 0.04129100418090821" rpy="0 0 0" />
+      <mass value="${mass_board}" />
+      <origin xyz="${mass_center_board}" rpy="0 0 0" />
       <inertia ixx="0.411139" iyy="0.524283" izz="0.881935" ixy="-0.000859" iyz="-0.000268" ixz="0.063417" />
     </inertial>
     <visual>
-      <origin xyz="0 0 0" rpy="0 0 0" />
+      <origin xyz="${position_board}" rpy="0 0 0" />
       <geometry>
         <mesh filename="package://waver_description/meshes/board_link.stl" scale="${scale}" />
@@ -101,5 +101,5 @@
     </visual>
     <collision>
-      <origin xyz="0 0 0" rpy="0 0 0" />
+      <origin xyz="${position_board}" rpy="0 0 0" />
       <geometry>
         <mesh filename="package://waver_description/meshes/board_link.stl" scale="${scale}" />
@@ -109,10 +109,10 @@
   <link name="oled_screen_link">
     <inertial>
-      <mass value="0.014091265350616076" />
-      <origin xyz="-6.735318456776441e-07 0.05096461868286133 0.048232952117919926" rpy="0 0 0" />
+      <mass value="${mass_screen}" />
+      <origin xyz="${mass_center_screen}" rpy="0 0 0" />
       <inertia ixx="0.002338" iyy="0.018383" izz="0.020177" ixy="-0.0" iyz="-3.9e-05" ixz="-0.0" />
     </inertial>
     <visual>
-      <origin xyz="0 0 0" rpy="0 0 0" />
+      <origin xyz="${position_screen}" rpy="0 0 0" />
       <geometry>
         <mesh filename="package://waver_description/meshes/oled_screen_link.stl" scale="${scale}" />
@@ -121,5 +121,5 @@
     </visual>
     <collision>
-      <origin xyz="0 0 0" rpy="0 0 0" />
+      <origin xyz="${position_screen}" rpy="0 0 0" />
       <geometry>
         <mesh filename="package://waver_description/meshes/oled_screen_link.stl" scale="${scale}" />
@@ -129,10 +129,10 @@
   <link name="wheel_back_left_link">
     <inertial>
-      <mass value="1.01701435808657" />
-      <origin xyz="0.06538582611083985 0.04859128189086914 0.004798986434936523" rpy="0 0 0" />
+      <mass value="${mass_wbl}" />
+      <origin xyz="${mass_center_wbl}" rpy="0 0 0" />
       <inertia ixx="9.903047" iyy="6.209714" izz="6.209755" ixy="2e-06" iyz="1.5e-05" ixz="5e-06" />
     </inertial>
     <visual>
-      <origin xyz="0 0 0" rpy="0 0 0" />
+      <origin xyz="${position_wbl}" rpy="0 0 0" />
       <geometry>
         <mesh filename="package://waver_description/meshes/wheel_back_left_link.stl" scale="${scale}" />
@@ -141,5 +141,5 @@
     </visual>
     <collision>
-      <origin xyz="0 0 0" rpy="0 0 0" />
+      <origin xyz="${position_wbl}" rpy="0 0 0" />
       <geometry>
         <mesh filename="package://waver_description/meshes/wheel_back_left_link.stl" scale="${scale}" />
@@ -149,10 +149,10 @@
   <link name="wheel_front_left_link">
     <inertial>
-      <mass value="1.0170155374515382" />
-      <origin xyz="0.06538582611083985 -0.048406845092773446 0.004799012184143066" rpy="0 0 0" />
+      <mass value="${mass_wfl}" />
+      <origin xyz="${mass_center_wfl}" rpy="0 0 0" />
       <inertia ixx="9.903064" iyy="6.20972" izz="6.20977" ixy="3e-06" iyz="9e-06" ixz="5e-06" />
     </inertial>
     <visual>
-      <origin xyz="0 0 0" rpy="0 0 0" />
+      <origin xyz="${position_wfl}" rpy="0 0 0" />
       <geometry>
         <mesh filename="package://waver_description/meshes/wheel_front_left_link.stl" scale="${scale}" />
@@ -161,5 +161,5 @@
     </visual>
     <collision>
-      <origin xyz="0 0 0" rpy="0 0 0" />
+      <origin xyz="${position_wfl}" rpy="0 0 0" />
       <geometry>
         <mesh filename="package://waver_description/meshes/wheel_front_left_link.stl" scale="${scale}" />
@@ -169,10 +169,10 @@
   <link name="wheel_front_right_link">
     <inertial>
-      <mass value="1.0170112199417978" />
-      <origin xyz="-0.06528724670410156 -0.048593093872070316 0.004798998355865478" rpy="0 0 0" />
+      <mass value="${mass_wfr}" />
+      <origin xyz="${mass_center_wfr}" rpy="0 0 0" />
       <inertia ixx="9.903034" iyy="6.2097" izz="6.209738" ixy="-7e-06" iyz="1e-05" ixz="6e-06" />
     </inertial>
     <visual>
-      <origin xyz="0 0 0" rpy="0 0 0" />
+      <origin xyz="${position_wfr}" rpy="0 0 0" />
       <geometry>
         <mesh filename="package://waver_description/meshes/wheel_front_right_link.stl" scale="${scale}" />
@@ -181,5 +181,5 @@
     </visual>
     <collision>
-      <origin xyz="0 0 0" rpy="0 0 0" />
+      <origin xyz="${position_wfr}" rpy="0 0 0" />
       <geometry>
         <mesh filename="package://waver_description/meshes/wheel_front_right_link.stl" scale="${scale}" />
@@ -189,10 +189,10 @@
   <link name="wheel_back_right_link">
     <inertial>
-      <mass value="1.0170123141691128" />
-      <origin xyz="-0.0652872543334961 0.04840502166748047 0.004799028396606446" rpy="0 0 0" />
+      <mass value="${mass_wbr}" />
+      <origin xyz="${mass_center_wbr}" rpy="0 0 0" />
       <inertia ixx="9.903051" iyy="6.209704" izz="6.209756" ixy="-7e-06" iyz="8e-06" ixz="5e-06" />
     </inertial>
     <visual>
-      <origin xyz="0 0 0" rpy="0 0 0" />
+      <origin xyz="${position_wbr}" rpy="0 0 0" />
       <geometry>
         <mesh filename="package://waver_description/meshes/wheel_back_right_link.stl" scale="${scale}" />
@@ -201,5 +201,5 @@
     </visual>
     <collision>
-      <origin xyz="0 0 0" rpy="0 0 0" />
+      <origin xyz="${position_wbr}" rpy="0 0 0" />
       <geometry>
         <mesh filename="package://waver_description/meshes/wheel_back_right_link.stl" scale="${scale}" />
@@ -220,46 +220,70 @@
   </joint>
   <joint name="top_acces_joint" type="fixed">
-    <origin xyz="0 0 0" rpy="0 0 0" />
+    <origin xyz="${mass_center_acces}" rpy="0 0 0" />
     <parent link="top_shell_link" />
     <child link="accessories_link" />
   </joint>
   <joint name="top_acces1_joint" type="fixed">
-    <origin xyz="0 0 0" rpy="0 0 0" />
+    <origin xyz="${mass_center_acces1}" rpy="0 0 0" />
     <parent link="top_shell_link" />
     <child link="accessories1_link" />
   </joint>
   <joint name="top_board_joint" type="fixed">
-    <origin xyz="0 0 0" rpy="0 0 0" />
+    <origin xyz="${mass_center_board}" rpy="0 0 0" />
     <parent link="top_shell_link" />
     <child link="board_link" />
   </joint>
   <joint name="top_screen_joint" type="fixed">
-    <origin xyz="0 0 0" rpy="0 0 0" />
+    <origin xyz="${mass_center_screen}" rpy="0 0 0" />
     <parent link="top_shell_link" />
     <child link="oled_screen_link" />
   </joint>
-  <joint name="base_wbl_joint" type="continuous">
-    <origin xyz="0 0 0" rpy="0 0 0" />
+  <joint name="wheel_back_left_joint" type="continuous">
+    <origin xyz="${mass_center_wbl}" rpy="0 0 0" />
     <parent link="base_link" />
     <child link="wheel_back_left_link" />
     <axis xyz="1 0 0" />
   </joint>
-  <joint name="base_wfl_joint" type="continuous">
-    <origin xyz="0 0 0" rpy="0 0 0" />
+  <joint name="wheel_front_left_joint" type="continuous">
+    <origin xyz="${mass_center_wfl}" rpy="0 0 0" />
     <parent link="base_link" />
     <child link="wheel_front_left_link" />
     <axis xyz="1 0 0" />
   </joint>
-  <joint name="base_wfr_joint" type="continuous">
-    <origin xyz="0 0 0" rpy="0 0 0" />
+  <joint name="wheel_front_right_joint" type="continuous">
+    <origin xyz="${mass_center_wfr}" rpy="0 0 0" />
     <parent link="base_link" />
     <child link="wheel_front_right_link" />
     <axis xyz="1 0 0" />
   </joint>
-  <joint name="base_wbr_joint" type="continuous">
-    <origin xyz="0 0 0" rpy="0 0 0" />
+  <joint name="wheel_back_right_joint" type="continuous">
+    <origin xyz="${mass_center_wbr}" rpy="0 0 0" />
     <parent link="base_link" />
     <child link="wheel_back_right_link" />
     <axis xyz="1 0 0" />
   </joint>
+  <gazebo>
+    <plugin name="skid_steer_drive_controller" filename="libgazebo_ros_skid_steer_drive.so">
+      <robotNamespace></robotNamespace>
+      <updateRate>100.0</updateRate>
+      <leftFrontJoint>wheel_front_left_joint</leftFrontJoint>
+      <rightFrontJoint>wheel_front_right_joint</rightFrontJoint>
+      <leftRearJoint>wheel_back_left_joint</leftRearJoint>
+      <rightRearJoint>wheel_back_right_joint</rightRearJoint>
+      <wheelSeparation>${wheel_separation}</wheelSeparation>
+      <wheelDiameter>${2*wheel_radius}</wheelDiameter>
+      <torque>10.0</torque>
+      <commandTopic>cmd_vel</commandTopic>
+      <odometryTopic>odom</odometryTopic>
+      <odometryFrame>odom</odometryFrame>
+      <robotBaseFrame>base_footprint</robotBaseFrame>
+      <publishWheelTF>true</publishWheelTF>
+      <publishOdom>true</publishOdom>
+      <publishWheelJointState>true</publishWheelJointState>
+      <covariance_x>0.0001</covariance_x>
+      <covariance_y>0.0001</covariance_y>
+      <covariance_yaw>0.01</covariance_yaw>
+      <broadcastTF>true</broadcastTF>
+    </plugin>
+  </gazebo>
 </robot>
