Commit message: fix: updated inertia and mass

File: waver_ws/src/waver_description/urdf/util.xacro (robot description, xacro)
@@ -22,5 +22,5 @@
     <xacro:property name="pos_y_acces" value="0.08693458557128907" />
     <xacro:property name="pos_z_acces" value="0.04861989974975586" />
-    <xacro:property name="mass_acces" value="0.017616158924187116" />
+    <xacro:property name="mass_acces" value="0.0017616158924187116" />
     <xacro:property name="mass_center_acces" value="${pos_x_acces} ${pos_y_acces} ${pos_z_acces}" />
     <xacro:property name="position_acces" value="${-pos_x_acces} ${-pos_y_acces} ${-pos_z_acces}" />
@@ -29,5 +29,5 @@
     <xacro:property name="pos_y_acces1" value="0.07360986328125002" />
     <xacro:property name="pos_z_acces1" value="0.035275302886962887" />
-    <xacro:property name="mass_acces1" value="0.021489822783274555" />
+    <xacro:property name="mass_acces1" value="0.0021489822783274555" />
     <xacro:property name="mass_center_acces1" value="${pos_x_acces1} ${pos_y_acces1} ${pos_z_acces1}" />
     <xacro:property name="position_acces1" value="${-pos_x_acces1} ${-pos_y_acces1} ${-pos_z_acces1}" />
@@ -36,5 +36,5 @@
     <xacro:property name="pos_y_board" value="0.009279213905334474" />
     <xacro:property name="pos_z_board" value="0.04129100418090821" />
-    <xacro:property name="mass_board" value="0.12365568710683028" />
+    <xacro:property name="mass_board" value="0.012365568710683028" />
     <xacro:property name="mass_center_board" value="${pos_x_board} ${pos_y_board} ${pos_z_board}" />
     <xacro:property name="position_board" value="${-pos_x_board} ${-pos_y_board} ${-pos_z_board}" />
@@ -43,5 +43,5 @@
     <xacro:property name="pos_y_screen" value="0.05096461868286133" />
     <xacro:property name="pos_z_screen" value="0.048232952117919926" />
-    <xacro:property name="mass_screen" value="0.014091265350616076" />
+    <xacro:property name="mass_screen" value="0.0014091265350616076" />
     <xacro:property name="mass_center_screen" value="${pos_x_screen} ${pos_y_screen} ${pos_z_screen}" />
     <xacro:property name="position_screen" value="${-pos_x_screen} ${-pos_y_screen} ${-pos_z_screen}" />

File: waver_ws/src/waver_description/urdf/waver.xacro (robot description, xacro)
@@ -51,5 +51,5 @@
       <mass value="${mass_acces}" />
       <origin xyz="${mass_center_acces}" rpy="0 0 0" />
-      <inertia ixx="2.2622278969724113e-06" iyy="7.36227380617578e-06" izz="7.362274117066844e-06" ixy="0.0" iyz="0.0" ixz="0.0" />
+      <inertia ixx="2.2622278969724113e-07" iyy="7.36227380617578e-07" izz="7.362274117066844e-07" ixy="0.0" iyz="0.0" ixz="0.0" />
     </inertial>
     <visual>
@@ -71,5 +71,5 @@
       <mass value="${mass_acces1}" />
       <origin xyz="${mass_center_acces1}" rpy="0 0 0" />
-      <inertia ixx="1.8160055789601745e-06" iyy="8.100907081280738e-06" izz="8.100806017664777e-06" ixy="0.0" iyz="0.0" ixz="0.0" />
+      <inertia ixx="1.8160055789601745e-07" iyy="8.100907081280738e-07" izz="8.100806017664777e-07" ixy="0.0" iyz="0.0" ixz="0.0" />
     </inertial>
     <visual>
@@ -91,5 +91,5 @@
       <mass value="${mass_board}" />
       <origin xyz="${mass_center_board}" rpy="0 0 0" />
-      <inertia ixx="5.313564367625195e-05" iyy="5.192849578266062e-05" izz="8.832425081682543e-05" ixy="0.0" iyz="0.0" ixz="0.0" />
+      <inertia ixx="5.313564367625195e-06" iyy="5.192849578266062e-06" izz="8.832425081682543e-06" ixy="0.0" iyz="0.0" ixz="0.0" />
     </inertial>
     <visual>
@@ -111,5 +111,5 @@
       <mass value="${mass_screen}" />
       <origin xyz="${mass_center_screen}" rpy="0 0 0" />
-      <inertia ixx="3.186534864702538e-07" iyy="2.5666330224105178e-06" izz="2.7215400443770056e-06" ixy="0.0" iyz="0.0" ixz="0.0" />
+      <inertia ixx="3.186534864702538e-08" iyy="2.5666330224105178e-07" izz="2.7215400443770056e-07" ixy="0.0" iyz="0.0" ixz="0.0" />
     </inertial>
     <visual>
