Commit message: fix: lidar orientation fixed

File: src/waver_description/urdf/lidar.xacro (robot description, xacro)
@@ -11,5 +11,5 @@
         </inertial>
         <visual>
-            <origin xyz="0 0 -0.027" rpy="0 0 0" />
+            <origin xyz="0 0 -0.027" rpy="0 0 ${pi/2}" />
             <geometry>
                 <mesh filename="package://waver_description/meshes/LD19.stl" scale="${scale}" />
@@ -18,5 +18,5 @@
         </visual>
         <collision>
-            <origin xyz="0 0 0" rpy="0 0 0" />
+            <origin xyz="0 0 -0.027" rpy="0 0 ${pi/2}" />
             <geometry>
                 <mesh filename="package://waver_description/meshes/LD19.stl" scale="${scale}" />
@@ -25,5 +25,5 @@
     </link>
     <joint name="lidar_joint" type="fixed">
-        <origin xyz="0 -0.04 ${base_to_top + 0.025}" rpy="0 0 0" />
+        <origin xyz="0 -0.04 ${base_to_top + 0.025}" rpy="0 0 ${-pi/2}" />
         <parent link="top_shell_link" />
         <child link="${lidar_link}" />

Commit message: fix: waver orientation fixed

File: src/waver_description/urdf/lidar.xacro (robot description, xacro)
@@ -25,5 +25,5 @@
     </link>
     <joint name="lidar_joint" type="fixed">
-        <origin xyz="0 -0.04 ${base_to_top + 0.025}" rpy="0 0 ${-pi/2}" />
+        <origin xyz="0.04 0 ${base_to_top + 0.025}" rpy="0 0 0" />
         <parent link="top_shell_link" />
         <child link="${lidar_link}" />

File: src/waver_description/urdf/util.xacro (robot description, xacro)
@@ -28,5 +28,6 @@
     <xacro:property name="mass_acces" value="0.0017616158924187116" />
     <xacro:property name="mass_center_acces" value="${pos_x_acces} ${pos_y_acces} ${pos_z_acces}" />
-    <xacro:property name="position_acces" value="${-pos_x_acces} ${-pos_y_acces} ${-pos_z_acces}" />
+    <xacro:property name="position_acces" value="${pos_y_acces} ${-pos_x_acces} ${-pos_z_acces}" />
+    <xacro:property name="positions_acces_joint" value="${-pos_y_acces} ${pos_x_acces} ${pos_z_acces}"/>
     <!-- Accessories1 specifications -->
     <xacro:property name="pos_x_acces1" value="-0.002510018587112427" />
@@ -35,5 +36,6 @@
     <xacro:property name="mass_acces1" value="0.0021489822783274555" />
     <xacro:property name="mass_center_acces1" value="${pos_x_acces1} ${pos_y_acces1} ${pos_z_acces1}" />
-    <xacro:property name="position_acces1" value="${-pos_x_acces1} ${-pos_y_acces1} ${-pos_z_acces1}" />
+    <xacro:property name="position_acces1" value="${pos_y_acces1} ${-pos_x_acces1} ${-pos_z_acces1}" />
+    <xacro:property name="positions_acces1_joint" value="${-pos_y_acces1} ${pos_x_acces1} ${pos_z_acces1}"/>
     <!-- Board speficications -->
     <xacro:property name="pos_x_board" value="-0.009815516471862793" />
@@ -42,5 +44,6 @@
     <xacro:property name="mass_board" value="0.012365568710683028" />
     <xacro:property name="mass_center_board" value="${pos_x_board} ${pos_y_board} ${pos_z_board}" />
-    <xacro:property name="position_board" value="${-pos_x_board} ${-pos_y_board} ${-pos_z_board}" />
+    <xacro:property name="position_board" value="${pos_y_board} ${-pos_x_board} ${-pos_z_board}" />
+    <xacro:property name="positions_board_joint" value="${-pos_y_board} ${pos_x_board} ${pos_z_board}"/>
     <!-- Oled Screen speficications -->
     <xacro:property name="pos_x_screen" value="-6.735318456776441e-07" />
@@ -49,5 +52,6 @@
     <xacro:property name="mass_screen" value="0.0014091265350616076" />
     <xacro:property name="mass_center_screen" value="${pos_x_screen} ${pos_y_screen} ${pos_z_screen}" />
-    <xacro:property name="position_screen" value="${-pos_x_screen} ${-pos_y_screen} ${-pos_z_screen}" />
+    <xacro:property name="position_screen" value="${pos_y_screen} ${-pos_x_screen} ${-pos_z_screen}" />
+    <xacro:property name="positions_screen_joint" value="${-pos_y_screen} ${pos_x_screen} ${pos_z_screen}"/>
     <!-- Wheels specifications -->
     <xacro:property name="wheel_separation" value="123e-3" />
@@ -59,5 +63,6 @@
     <xacro:property name="mass_wbl" value="1.01701435808657" />
     <xacro:property name="mass_center_wbl" value="${pos_x_wbl} ${pos_y_wbl} ${pos_z_wbl}" />
-    <xacro:property name="position_wbl" value="${-pos_x_wbl} ${-pos_y_wbl} ${-pos_z_wbl}" />
+    <xacro:property name="position_wbl" value="${pos_y_wbl} ${-pos_x_wbl} ${-pos_z_wbl}" />
+    <xacro:property name="position_wbl_joint" value="${-pos_y_wbl} ${pos_x_wbl} ${pos_z_wbl}"/>
     <!-- WFL specifications -->
     <xacro:property name="pos_x_wfl" value="0.06538582611083985" />
@@ -66,5 +71,6 @@
     <xacro:property name="mass_wfl" value="1.0170155374515382" />
     <xacro:property name="mass_center_wfl" value="${pos_x_wfl} ${pos_y_wfl} ${pos_z_wfl}" />
-    <xacro:property name="position_wfl" value="${-pos_x_wfl} ${-pos_y_wfl} ${-pos_z_wfl}" />
+    <xacro:property name="position_wfl" value="${pos_y_wfl} ${-pos_x_wfl} ${-pos_z_wfl}" />
+    <xacro:property name="position_wfl_joint" value="${-pos_y_wfl} ${pos_x_wfl} ${pos_z_wfl}"/>
     <!-- WFR specifications -->
     <xacro:property name="pos_x_wfr" value="-0.06528724670410156" />
@@ -73,5 +79,6 @@
     <xacro:property name="mass_wfr" value="1.0170112199417978" />
     <xacro:property name="mass_center_wfr" value="${pos_x_wfr} ${pos_y_wfr} ${pos_z_wfr}" />
-    <xacro:property name="position_wfr" value="${-pos_x_wfr} ${-pos_y_wfr} ${-pos_z_wfr}" />
+    <xacro:property name="position_wfr" value="${pos_y_wfr} ${-pos_x_wfr} ${-pos_z_wfr}" />
+    <xacro:property name="position_wfr_joint" value="${-pos_y_wfr} ${pos_x_wfr} ${pos_z_wfr}"/>
     <!-- WBR specifications -->
     <xacro:property name="pos_x_wbr" value="-0.0652872543334961" />
@@ -80,5 +87,6 @@
     <xacro:property name="mass_wbr" value="1.0170123141691128" />
     <xacro:property name="mass_center_wbr" value="${pos_x_wbr} ${pos_y_wbr} ${pos_z_wbr}" />
-    <xacro:property name="position_wbr" value="${-pos_x_wbr} ${-pos_y_wbr} ${-pos_z_wbr}" />
+    <xacro:property name="position_wbr" value="${pos_y_wbr} ${-pos_x_wbr} ${-pos_z_wbr}" />
+    <xacro:property name="position_wbr_joint" value="${-pos_y_wbr} ${pos_x_wbr} ${pos_z_wbr}"/>
     <!-- Lidar specifications -->
     <xacro:property name="mass_lidar" value="0.05" />

File: src/waver_description/urdf/waver.xacro (robot description, xacro)
@@ -11,9 +11,9 @@
     <inertial>
       <mass value="${mass_base}" />
-      <origin xyz="${mass_center_base}" rpy="0 0 0" />
+      <origin xyz="${mass_center_base}" rpy="0 0 ${pi/2}" />
       <inertia ixx="0.0008255973835920386" iyy="0.0005293282898445326" izz="0.0013315199498696443" ixy="0.0" iyz="0.0" ixz="0.0" />
     </inertial>
     <visual>
-      <origin xyz="0 0 0" rpy="0 0 0" />
+      <origin xyz="0 0 0" rpy="0 0 ${pi/2}" />
       <geometry>
         <mesh filename="package://waver_description/meshes/base_link.stl" scale="${scale}" />
@@ -22,5 +22,5 @@
     </visual>
     <collision>
-      <origin xyz="0 0 0" rpy="0 0 0" />
+      <origin xyz="0 0 0" rpy="0 0 ${pi/2}" />
       <geometry>
         <mesh filename="package://waver_description/meshes/base_link.stl" scale="${scale}" />
@@ -31,9 +31,9 @@
     <inertial>
       <mass value="${mass_top}" />
-      <origin xyz="${mass_center_top}" rpy="0 0 0" />
+      <origin xyz="${mass_center_top}" rpy="0 0 ${pi/2}" />
       <inertia ixx="0.0022122780308922725" iyy="0.0018048674350663336" izz="0.003659349844340526" ixy="0.0" iyz="0.0" ixz="0.0" />
     </inertial>
     <visual>
-      <origin xyz="0 0 0" rpy="0 0 0" />
+      <origin xyz="0 0 0" rpy="0 0 ${pi/2}" />
       <geometry>
         <mesh filename="package://waver_description/meshes/top_shell_link.stl" scale="${scale}" />
@@ -42,5 +42,5 @@
     </visual>
     <collision>
-      <origin xyz="0 0 0" rpy="0 0 0" />
+      <origin xyz="0 0 0" rpy="0 0 ${pi/2}" />
       <geometry>
         <mesh filename="package://waver_description/meshes/top_shell_link.stl" scale="${scale}" />
@@ -51,9 +51,9 @@
     <inertial>
       <mass value="${mass_acces}" />
-      <origin xyz="${mass_center_acces}" rpy="0 0 0" />
+      <origin xyz="${mass_center_acces}" rpy="0 0 ${pi/2}" />
       <inertia ixx="2.2622278969724113e-07" iyy="7.36227380617578e-07" izz="7.362274117066844e-07" ixy="0.0" iyz="0.0" ixz="0.0" />
     </inertial>
     <visual>
-      <origin xyz="${position_acces}" rpy="0 0 0" />
+      <origin xyz="${position_acces}" rpy="0 0 ${pi/2}" />
       <geometry>
         <mesh filename="package://waver_description/meshes/accessories_link.stl" scale="${scale}" />
@@ -62,5 +62,5 @@
     </visual>
     <collision>
-      <origin xyz="${position_acces}" rpy="0 0 0" />
+      <origin xyz="${position_acces}" rpy="0 0 ${pi/2}" />
       <geometry>
         <mesh filename="package://waver_description/meshes/accessories_link.stl" scale="${scale}" />
@@ -71,9 +71,9 @@
     <inertial>
       <mass value="${mass_acces1}" />
-      <origin xyz="${mass_center_acces1}" rpy="0 0 0" />
+      <origin xyz="${mass_center_acces1}" rpy="0 0 ${pi/2}" />
       <inertia ixx="1.8160055789601745e-07" iyy="8.100907081280738e-07" izz="8.100806017664777e-07" ixy="0.0" iyz="0.0" ixz="0.0" />
     </inertial>
     <visual>
-      <origin xyz="${position_acces1}" rpy="0 0 0" />
+      <origin xyz="${position_acces1}" rpy="0 0 ${pi/2}" />
       <geometry>
         <mesh filename="package://waver_description/meshes/accessories1_link.stl" scale="${scale}" />
@@ -82,5 +82,5 @@
     </visual>
     <collision>
-      <origin xyz="${position_acces1}" rpy="0 0 0" />
+      <origin xyz="${position_acces1}" rpy="0 0 ${pi/2}" />
       <geometry>
         <mesh filename="package://waver_description/meshes/accessories1_link.stl" scale="${scale}" />
@@ -91,9 +91,9 @@
     <inertial>
       <mass value="${mass_board}" />
-      <origin xyz="${mass_center_board}" rpy="0 0 0" />
+      <origin xyz="${mass_center_board}" rpy="0 0 ${pi/2}" />
       <inertia ixx="5.313564367625195e-06" iyy="5.192849578266062e-06" izz="8.832425081682543e-06" ixy="0.0" iyz="0.0" ixz="0.0" />
     </inertial>
     <visual>
-      <origin xyz="${position_board}" rpy="0 0 0" />
+      <origin xyz="${position_board}" rpy="0 0 ${pi/2}" />
       <geometry>
         <mesh filename="package://waver_description/meshes/board_link.stl" scale="${scale}" />
@@ -102,5 +102,5 @@
     </visual>
     <collision>
-      <origin xyz="${position_board}" rpy="0 0 0" />
+      <origin xyz="${position_board}" rpy="0 0 ${pi/2}" />
       <geometry>
         <mesh filename="package://waver_description/meshes/board_link.stl" scale="${scale}" />
@@ -111,9 +111,9 @@
     <inertial>
       <mass value="${mass_screen}" />
-      <origin xyz="${mass_center_screen}" rpy="0 0 0" />
+      <origin xyz="${mass_center_screen}" rpy="0 0 ${pi/2}" />
       <inertia ixx="3.186534864702538e-08" iyy="2.5666330224105178e-07" izz="2.7215400443770056e-07" ixy="0.0" iyz="0.0" ixz="0.0" />
     </inertial>
     <visual>
-      <origin xyz="${position_screen}" rpy="0 0 0" />
+      <origin xyz="${position_screen}" rpy="0 0 ${pi/2}" />
       <geometry>
         <mesh filename="package://waver_description/meshes/oled_screen_link.stl" scale="${scale}" />
@@ -122,5 +122,5 @@
     </visual>
     <collision>
-      <origin xyz="${position_screen}" rpy="0 0 0" />
+      <origin xyz="${position_screen}" rpy="0 0 ${pi/2}" />
       <geometry>
         <mesh filename="package://waver_description/meshes/oled_screen_link.stl" scale="${scale}" />
@@ -131,9 +131,9 @@
     <inertial>
       <mass value="${mass_wbl}" />
-      <origin xyz="0 0 0" rpy="0 0 0" />
+      <origin xyz="0 0 0" rpy="0 0 ${pi/2}" />
       <inertia ixx="0.0011153598236428852" iyy="0.0007115715200341761" izz="0.0007099489264864056" ixy="0.0" iyz="0.0" ixz="0.0" />
     </inertial>
     <visual>
-      <origin xyz="${position_wbl}" rpy="0 0 0" />
+      <origin xyz="${position_wbl}" rpy="0 0 ${pi/2}" />
       <geometry>
         <mesh filename="package://waver_description/meshes/wheel_back_left_link.stl" scale="${scale}" />
@@ -142,5 +142,5 @@
     </visual>
     <collision>
-      <origin xyz="${position_wbl}" rpy="0 0 0" />
+      <origin xyz="${position_wbl}" rpy="0 0 ${pi/2}" />
       <geometry>
         <mesh filename="package://waver_description/meshes/wheel_back_left_link.stl" scale="${scale}" />
@@ -151,9 +151,9 @@
     <inertial>
       <mass value="${mass_wfl}" />
-      <origin xyz="0 0 0" rpy="0 0 0" />
+      <origin xyz="0 0 0" rpy="0 0 ${pi/2}" />
       <inertia ixx="0.0011153873944048257" iyy="0.0007115715200341761" izz="0.0007099764972483459" ixy="0.0" iyz="0.0" ixz="0.0" />
     </inertial>
     <visual>
-      <origin xyz="${position_wfl}" rpy="0 0 0" />
+      <origin xyz="${position_wfl}" rpy="0 0 ${pi/2}" />
       <geometry>
         <mesh filename="package://waver_description/meshes/wheel_front_left_link.stl" scale="${scale}" />
@@ -162,5 +162,5 @@
     </visual>
     <collision>
-      <origin xyz="${position_wfl}" rpy="0 0 0" />
+      <origin xyz="${position_wfl}" rpy="0 0 ${pi/2}" />
       <geometry>
         <mesh filename="package://waver_description/meshes/wheel_front_left_link.stl" scale="${scale}" />
@@ -171,9 +171,9 @@
     <inertial>
       <mass value="${mass_wfr}" />
-      <origin xyz="0 0 0" rpy="0 0 0" />
+      <origin xyz="0 0 0" rpy="0 0 ${pi/2}" />
       <inertia ixx="0.0011153598236428852" iyy="0.0007115715475157099" izz="0.0007099489539679392" ixy="0.0" iyz="0.0" ixz="0.0" />
     </inertial>
     <visual>
-      <origin xyz="${position_wfr}" rpy="0 0 0" />
+      <origin xyz="${position_wfr}" rpy="0 0 ${pi/2}" />
       <geometry>
         <mesh filename="package://waver_description/meshes/wheel_front_right_link.stl" scale="${scale}" />
@@ -182,5 +182,5 @@
     </visual>
     <collision>
-      <origin xyz="${position_wfr}" rpy="0 0 0" />
+      <origin xyz="${position_wfr}" rpy="0 0 ${pi/2}" />
       <geometry>
         <mesh filename="package://waver_description/meshes/wheel_front_right_link.stl" scale="${scale}" />
@@ -191,9 +191,9 @@
     <inertial>
       <mass value="${mass_wbr}" />
-      <origin xyz="0 0 0" rpy="0 0 0" />
+      <origin xyz="0 0 0" rpy="0 0 ${pi/2}" />
       <inertia ixx="0.0011153873944048257" iyy="0.0007115715475157099" izz="0.0007099765247298796" ixy="0.0" iyz="0.0" ixz="0.0" />
     </inertial>
     <visual>
-      <origin xyz="${position_wbr}" rpy="0 0 0" />
+      <origin xyz="${position_wbr}" rpy="0 0 ${pi/2}" />
       <geometry>
         <mesh filename="package://waver_description/meshes/wheel_back_right_link.stl" scale="${scale}" />
@@ -202,5 +202,5 @@
     </visual>
     <collision>
-      <origin xyz="${position_wbr}" rpy="0 0 0" />
+      <origin xyz="${position_wbr}" rpy="0 0 ${pi/2}" />
       <geometry>
         <mesh filename="package://waver_description/meshes/wheel_back_right_link.stl" scale="${scale}" />
@@ -221,46 +221,46 @@
   </joint>
   <joint name="top_acces_joint" type="fixed">
-    <origin xyz="${mass_center_acces}" rpy="0 0 0" />
+    <origin xyz="${positions_acces_joint}" rpy="0 0 0" />
     <parent link="top_shell_link" />
     <child link="accessories_link" />
   </joint>
-  <joint name="top_acces1_joint" type="fixed">
-    <origin xyz="${mass_center_acces1}" rpy="0 0 0" />
+<joint name="top_acces1_joint" type="fixed">
+    <origin xyz="${positions_acces1_joint}" rpy="0 0 0" />
     <parent link="top_shell_link" />
     <child link="accessories1_link" />
   </joint>
   <joint name="top_board_joint" type="fixed">
-    <origin xyz="${mass_center_board}" rpy="0 0 0" />
+    <origin xyz="${positions_board_joint}" rpy="0 0 0" />
     <parent link="top_shell_link" />
     <child link="board_link" />
   </joint>
   <joint name="top_screen_joint" type="fixed">
-    <origin xyz="${mass_center_screen}" rpy="0 0 0" />
+    <origin xyz="${positions_screen_joint}" rpy="0 0 0" />
     <parent link="top_shell_link" />
     <child link="oled_screen_link" />
   </joint>
   <joint name="wheel_back_left_joint" type="continuous">
-    <origin xyz="${mass_center_wbl}" rpy="0 0 0" />
+    <origin xyz="${position_wbl_joint}" rpy="0 0 0" />
     <parent link="base_link" />
     <child link="wheel_back_left_link" />
-    <axis xyz="1 0 0" />
+    <axis xyz="0 1 0" />
   </joint>
   <joint name="wheel_front_left_joint" type="continuous">
-    <origin xyz="${mass_center_wfl}" rpy="0 0 0" />
+    <origin xyz="${position_wfl_joint}" rpy="0 0 0" />
     <parent link="base_link" />
     <child link="wheel_front_left_link" />
-    <axis xyz="1 0 0" />
+    <axis xyz="0 1 0" />
   </joint>
   <joint name="wheel_front_right_joint" type="continuous">
-    <origin xyz="${mass_center_wfr}" rpy="0 0 0" />
+    <origin xyz="${position_wfr_joint}" rpy="0 0 0" />
     <parent link="base_link" />
     <child link="wheel_front_right_link" />
-    <axis xyz="1 0 0" />
+    <axis xyz="0 1 0" />
   </joint>
   <joint name="wheel_back_right_joint" type="continuous">
-    <origin xyz="${mass_center_wbr}" rpy="0 0 0" />
+    <origin xyz="${position_wbr_joint}" rpy="0 0 0" />
     <parent link="base_link" />
     <child link="wheel_back_right_link" />
-    <axis xyz="1 0 0" />
+    <axis xyz="0 1 0" />
   </joint>
   <gazebo>
@@ -278,5 +278,5 @@
       <odometryTopic>odom</odometryTopic>
       <odometryFrame>odom</odometryFrame>
-      <robotBaseFrame>base_footprint</robotBaseFrame>
+      <robotBaseFrame>base_link</robotBaseFrame>
       <publishWheelTF>true</publishWheelTF>
       <publishOdom>true</publishOdom>
