Commit message: feat: imu added

File: waver_description/urdf/util.xacro (robot description, xacro)
@@ -38,12 +38,12 @@
     <xacro:property name="position_acces1" value="${pos_y_acces1} ${-pos_x_acces1} ${-pos_z_acces1}" />
     <xacro:property name="positions_acces1_joint" value="${-pos_y_acces1} ${pos_x_acces1} ${pos_z_acces1}"/>
-    <!-- Board speficications -->
-    <xacro:property name="pos_x_board" value="-0.009815516471862793" />
-    <xacro:property name="pos_y_board" value="0.009279213905334474" />
-    <xacro:property name="pos_z_board" value="0.04129100418090821" />
-    <xacro:property name="mass_board" value="0.012365568710683028" />
-    <xacro:property name="mass_center_board" value="${pos_x_board} ${pos_y_board} ${pos_z_board}" />
-    <xacro:property name="position_board" value="${pos_y_board} ${-pos_x_board} ${-pos_z_board}" />
-    <xacro:property name="positions_board_joint" value="${-pos_y_board} ${pos_x_board} ${pos_z_board}"/>
+    <!-- IMU speficications -->
+    <xacro:property name="pos_x_imu" value="-0.009815516471862793" />
+    <xacro:property name="pos_y_imu" value="0.009279213905334474" />
+    <xacro:property name="pos_z_imu" value="0.04129100418090821" />
+    <xacro:property name="mass_imu" value="0.012365568710683028" />
+    <xacro:property name="mass_center_imu" value="${pos_x_imu} ${pos_y_imu} ${pos_z_imu}" />
+    <xacro:property name="position_imu" value="${pos_y_imu} ${-pos_x_imu} ${-pos_z_imu}" />
+    <xacro:property name="positions_imu_joint" value="${-pos_y_imu} ${pos_x_imu} ${pos_z_imu}"/>
     <!-- Oled Screen speficications -->
     <xacro:property name="pos_x_screen" value="-6.735318456776441e-07" />

File: waver_description/urdf/waver.gazebo.xacro (robot description, xacro)
@@ -26,5 +26,5 @@
     <material>Gazebo/Black</material>
   </gazebo>
-  <gazebo reference="board_link">
+  <gazebo reference="imu_link">
     <mu1>0.2</mu1>
     <mu2>0.2</mu2>

File: waver_description/urdf/waver.xacro (robot description, xacro)
@@ -6,4 +6,5 @@
   <xacro:include filename="$(find waver_description)/urdf/waver.gazebo.xacro" />
   <xacro:include filename="$(find waver_description)/urdf/lidar.xacro" />
+  <xacro:include filename="$(find waver_description)/urdf/imu.xacro" />
   <!-- ******************************* Links ******************************* -->
   <link name="base_footprint"></link>
@@ -85,24 +86,4 @@
       <geometry>
         <mesh filename="package://waver_description/meshes/accessories1_link.stl" scale="${scale}" />
-      </geometry>
-    </collision>
-  </link>
-  <link name="board_link">
-    <inertial>
-      <mass value="${mass_board}" />
-      <origin xyz="${mass_center_board}" rpy="0 0 ${pi/2}" />
-      <inertia ixx="5.313564367625195e-06" iyy="5.192849578266062e-06" izz="8.832425081682543e-06" ixy="0.0" iyz="0.0" ixz="0.0" />
-    </inertial>
-    <visual>
-      <origin xyz="${position_board}" rpy="0 0 ${pi/2}" />
-      <geometry>
-        <mesh filename="package://waver_description/meshes/board_link.stl" scale="${scale}" />
-      </geometry>
-      <xacro:dark_green_material />
-    </visual>
-    <collision>
-      <origin xyz="${position_board}" rpy="0 0 ${pi/2}" />
-      <geometry>
-        <mesh filename="package://waver_description/meshes/board_link.stl" scale="${scale}" />
       </geometry>
     </collision>
@@ -230,9 +211,4 @@
     <child link="accessories1_link" />
   </joint>
-  <joint name="top_board_joint" type="fixed">
-    <origin xyz="${positions_board_joint}" rpy="0 0 0" />
-    <parent link="top_shell_link" />
-    <child link="board_link" />
-  </joint>
   <joint name="top_screen_joint" type="fixed">
     <origin xyz="${positions_screen_joint}" rpy="0 0 0" />
